Commit message: only add the plate model

File: src/rm_robot/rm_65_description/urdf/rm_65.urdf.xacro (robot description, xacro)
@@ -5,4 +5,5 @@
   <link name="dummy">
   </link>
+  <!--######################################################################-->
   <link
     name="base_link">
@@ -55,4 +56,5 @@
     <child link="base_link" />
   </joint>
+  <!--######################################################################-->
   <link
     name="Link1">
@@ -114,4 +116,5 @@
 	<dynamics damping="50" friction="1"/>
   </joint>
+  <!--######################################################################-->
   <link
     name="Link2">
@@ -173,4 +176,5 @@
 	<dynamics damping="50" friction="1"/>
   </joint>
+  <!--######################################################################-->
   <link
     name="Link3">
@@ -232,4 +236,5 @@
 	<dynamics damping="50" friction="1"/>
   </joint>
+  <!--######################################################################-->
   <link
     name="Link4">
@@ -291,4 +296,5 @@
 	<dynamics damping="50" friction="1"/>
   </joint>
+  <!--######################################################################-->
   <link
     name="Link5">
@@ -350,4 +356,5 @@
 	<dynamics damping="50" friction="1"/>
   </joint>
+  <!--######################################################################-->
   <link
     name="Link6">
@@ -409,4 +416,60 @@
 	<dynamics damping="50" friction="1"/>
   </joint>
+  <!-- This URDF was automatically created by SolidWorks to URDF Exporter! Originally created by Stephen Brawner (brawner@gmail.com)
+     Commit Version: 1.5.1-0-g916b5db  Build Version: 1.5.7152.31018
+     For more information, please see http://wiki.ros.org/sw_urdf_exporter -->
+  <link
+    name="plate">
+    <inertial>
+      <origin
+        xyz="0.04582 -2.25539999752262E-10 0.004046"
+        rpy="0 0 0" />
+      <mass
+        value="0.051308" />
+      <inertia
+        ixx="1.5915E-05"
+        ixy="2.51849999912398E-14"
+        ixz="1.4307E-07"
+        iyy="8.6534E-05"
+        iyz="4.91220000094025E-12"
+        izz="0.00010189" />
+    </inertial>
+    <visual>
+      <origin
+        xyz="0 0 0"
+        rpy="1.5707963267949 0 0" />
+      <geometry>
+        <mesh
+          filename="package://rm_65_description/meshes/plate.STL" />
+      </geometry>
+      <material
+        name="">
+        <color
+          rgba="1 1 1 1" />
+      </material>
+    </visual>
+    <collision>
+      <origin
+        xyz="0 0 0"
+        rpy="1.5707963267949 0 0" />
+      <geometry>
+        <mesh
+          filename="package://rm_65_description/meshes/plate.STL" />
+      </geometry>
+    </collision>
+  </link>
+  <joint
+    name="joint7"
+    type="fixed">
+    <origin
+      xyz="0 0 0"
+      rpy="0 0 3.1416" />
+    <parent
+      link="Link6" />
+    <child
+      link="plate" />
+    <dynamics damping="50" friction="1"/>
+  </joint>
+  <!--######################################################################-->
   <!-- Transmissions for ROS Control -->
   <xacro:macro name="transmission_block" params="joint_name">

Commit message: the URDF without gripper

File: src/rm_robot/rm_65_description/urdf/rm_65.urdf.xacro (robot description, xacro)
@@ -51,4 +51,5 @@
     <kp value="100000000.0"/>
     <kd value="1.0"/>
+    <material>Gazebo/Blue<material/>
   </gazebo>
   <joint name="dummy_joint" type="fixed">
@@ -416,4 +417,5 @@
 	<dynamics damping="50" friction="1"/>
   </joint>
+  <!--######################################################################-->
   <!-- This URDF was automatically created by SolidWorks to URDF Exporter! Originally created by Stephen Brawner (brawner@gmail.com)
      Commit Version: 1.5.1-0-g916b5db  Build Version: 1.5.7152.31018
@@ -471,4 +473,17 @@
     <dynamics damping="50" friction="1"/>
   </joint>
+  <!--######################################################################-->
+  <!-- plate -->
+  <xacro:arg name="use_nominal_extrinsics" default="false"/>
+  <xacro:arg name="add_plug" default="false" />
+  <xacro:arg name="use_mesh" default="true" />
+  <xacro:include filename="$(find realsense2_description)/urdf/_d435.urdf.xacro" />
+  <xacro:sensor_d435 parent="plate" use_nominal_extrinsics="$(arg use_nominal_extrinsics)" add_plug="$(arg add_plug)" use_mesh="$(arg use_mesh)">
+    <origin xyz="0.08 0 0.0185" rpy="0 -1.5708 3.1416"/>
+    <!-- <origin xyz="0.0925 0 0.008" rpy="0 -1.5708 0"/> -->
+  </xacro:sensor_d435>
+  <!--######################################################################-->
+  <!-- gripper -->
+  <!-- <xacro:include filename="$(find rm_65_description)/urdf/rm_65.gazebo.xacro"/> -->
   <!--######################################################################-->
   <!-- Transmissions for ROS Control -->

Commit message: with gripper. the d435 is the old version

File: src/rm_robot/rm_65_description/urdf/rm_65.urdf.xacro (robot description, xacro)
@@ -51,5 +51,4 @@
     <kp value="100000000.0"/>
     <kd value="1.0"/>
-    <material>Gazebo/Blue<material/>
   </gazebo>
   <joint name="dummy_joint" type="fixed">
@@ -486,4 +485,17 @@
   <!-- gripper -->
   <!-- <xacro:include filename="$(find rm_65_description)/urdf/rm_65.gazebo.xacro"/> -->
+  <xacro:include filename="$(find rm_65_description)/urdf/jawasm1.urdf" />
+  <joint
+    name="joint8"
+    type="fixed">
+    <origin
+      xyz="-0.0125 0 ${0.0535-0.0099185365078758+0.008}"
+      rpy="0 -1.5708 0" />
+    <parent
+      link="plate" />
+    <child
+      link="gripper_base_link" />
+    <dynamics damping="50" friction="1"/>
+  </joint>
   <!--######################################################################-->
   <!-- Transmissions for ROS Control -->
@@ -506,5 +518,5 @@
   <xacro:transmission_block joint_name="joint5"/>
   <xacro:transmission_block joint_name="joint6"/>
-  <!-- ros_control plugin -->
+  <!-- gazebo controller plugin for arm -->
   <gazebo>
     <plugin name="gazebo_ros_control" filename="libgazebo_ros_control.so">
@@ -514,3 +526,4 @@
     </plugin>
   </gazebo>
+  <!-- gazebo controller plugin for gripper -->
 </robot>
