Commit message: created rm_moveit_config without catkin build

File: src/rm_robot/rm_65_description/urdf/jawasm1.urdf.xacro (robot description, xacro)
@@ -1,4 +1,4 @@
-<robot
-  name="jawasm1">
+<?xml version="1.0" encoding="utf-8"?>
+<robot name="jawasm1" xmlns:xacro="http://www.ros.org/wiki/xacro">
   <link
     name="gripper_base_link">

File: src/rm_robot/rm_65_description/urdf/rm_65.urdf.xacro (robot description, xacro)
@@ -420,4 +420,5 @@
      Commit Version: 1.5.1-0-g916b5db  Build Version: 1.5.7152.31018
      For more information, please see http://wiki.ros.org/sw_urdf_exporter -->
+  <!-- plate -->
   <link
     name="plate">
@@ -473,5 +474,10 @@
   </joint>
   <!--######################################################################-->
-  <!-- plate -->
+  <!-- realsense d435 with gazebo simulation    joint8 -->
+  <xacro:include filename="$(find realsense_ros_gazebo)/xacro/depthcam.xacro"/>
+  <xacro:realsense_d435 sensor_name="d435" parent_link="plate" rate="10">
+    <origin rpy="0 -1.5708 3.1416" xyz="0.08 0 0.0185"/>
+  </xacro:realsense_d435>
+  <!--
   <xacro:arg name="use_nominal_extrinsics" default="false"/>
   <xacro:arg name="add_plug" default="false" />
@@ -480,15 +486,16 @@
   <xacro:sensor_d435 parent="plate" use_nominal_extrinsics="$(arg use_nominal_extrinsics)" add_plug="$(arg add_plug)" use_mesh="$(arg use_mesh)">
     <origin xyz="0.08 0 0.0185" rpy="0 -1.5708 3.1416"/>
-    <!-- <origin xyz="0.0925 0 0.008" rpy="0 -1.5708 0"/> -->
+    <origin xyz="0.0925 0 0.008" rpy="0 -1.5708 0"/>
   </xacro:sensor_d435>
+  -->
   <!--######################################################################-->
   <!-- gripper -->
   <!-- <xacro:include filename="$(find rm_65_description)/urdf/rm_65.gazebo.xacro"/> -->
-  <xacro:include filename="$(find rm_65_description)/urdf/jawasm1.urdf" />
-  <joint
-    name="joint8"
+  <xacro:include filename="$(find rm_65_description)/urdf/jawasm1.urdf.xacro" />
+  <joint
+    name="joint9"
     type="fixed">
     <origin
-      xyz="-0.0125 0 ${0.0535-0.0099185365078758+0.008}"
+      xyz="-0.0125 0 0.0516"
       rpy="0 -1.5708 0" />
     <parent
@@ -496,9 +503,9 @@
     <child
       link="gripper_base_link" />
-    <dynamics damping="50" friction="1"/>
+    <dynamics damping="50" friction="1" />
   </joint>
   <!--######################################################################-->
   <!-- Transmissions for ROS Control -->
-  <xacro:macro name="transmission_block" params="joint_name">
+  <xacro:macro name="transmission_block" params="joint_name" >
     <transmission name="tran1">
       <type>transmission_interface/SimpleTransmission</type>
@@ -518,8 +525,12 @@
   <xacro:transmission_block joint_name="joint5"/>
   <xacro:transmission_block joint_name="joint6"/>
+  <xacro:transmission_block joint_name="gripper_Link1"/>
+  <xacro:transmission_block joint_name="gripper_Link2"/>
+  <xacro:transmission_block joint_name="gripper_Link11"/>
+  <xacro:transmission_block joint_name="gripper_Link22"/>
   <!-- gazebo controller plugin for arm -->
   <gazebo>
     <plugin name="gazebo_ros_control" filename="libgazebo_ros_control.so">
-      <robotNamespace>/arm</robotNamespace>
+      <robotNamespace>/</robotNamespace>
       <robotSimType>gazebo_ros_control/DefaultRobotHWSim</robotSimType>
       <legacyModeNS>true</legacyModeNS>

Commit message: the xacro error

File: src/rm_robot/rm_65_description/urdf/jawasm1.urdf.xacro (robot description, xacro)
@@ -8,5 +8,5 @@
         rpy="0 0 0" />
       <mass
-        value="0.105853592307918" />
+        value="0.000001" />
       <inertia
         ixx="3.93795927851199E-05"
@@ -48,5 +48,5 @@
         rpy="0 0 0" />
       <mass
-        value="0.00647716099397792" />
+        value="0.000001" />
       <inertia
         ixx="2.95068972140683E-07"
@@ -106,5 +106,5 @@
         rpy="0 0 0" />
       <mass
-        value="0.0127543420299361" />
+        value="0.000001" />
       <inertia
         ixx="5.68538478020233E-07"
@@ -164,5 +164,5 @@
         rpy="0 0 0" />
       <mass
-        value="0.00647716099397793" />
+        value="0.000001" />
       <inertia
         ixx="2.95068972140683E-07"
@@ -222,5 +222,5 @@
         rpy="0 0 0" />
       <mass
-        value="0.0127543420299362" />
+        value="0.000001" />
       <inertia
         ixx="5.68538478020238E-07"

File: src/rm_robot/rm_65_description/urdf/rm_65.urdf.xacro (robot description, xacro)
@@ -5,20 +5,20 @@
   <link name="dummy">
   </link>
-  <!--######################################################################-->
+  <!-- base_link -->
   <link
     name="base_link">
     <inertial>
       <origin
-        xyz="-0.000433277303987328 -3.54664423471128E-05 0.0599427668933796"
+        xyz="0 0 0"
         rpy="0 0 0" />
       <mass
         value="14" />
       <inertia
-        ixx="0.0017261110801622"
-        ixy="2.52746264980217E-06"
-        ixz="-3.67690303614961E-05"
-        iyy="0.00170987405835604"
-        iyz="1.67996364994424E-06"
-        izz="0.000904023422915791" />
+        ixx="0.01"
+        ixy="0"
+        ixz="0"
+        iyy="0.01"
+        iyz="0"
+        izz="0.01" />
     </inertial>
     <visual>
@@ -56,5 +56,5 @@
     <child link="base_link" />
   </joint>
-  <!--######################################################################-->
+  <!-- Link1 -->
   <link
     name="Link1">
@@ -116,5 +116,5 @@
 	<dynamics damping="50" friction="1"/>
   </joint>
-  <!--######################################################################-->
+  <!-- Link2 -->
   <link
     name="Link2">
@@ -124,5 +124,5 @@
         rpy="0 0 0" />
       <mass
-        value="0.864175046869043" />
+        value="0.013" />
       <inertia
         ixx="0.00089150298478414"
@@ -176,5 +176,5 @@
 	<dynamics damping="50" friction="1"/>
   </joint>
-  <!--######################################################################-->
+  <!-- Link3 -->
   <link
     name="Link3">
@@ -184,5 +184,5 @@
         rpy="0 0 0" />
       <mass
-        value="0.289633681624654" />
+        value="0.013" />
       <inertia
         ixx="0.00063737100450158"
@@ -236,5 +236,5 @@
 	<dynamics damping="50" friction="1"/>
   </joint>
-  <!--######################################################################-->
+  <!-- Link4 -->
   <link
     name="Link4">
@@ -244,5 +244,5 @@
         rpy="0 0 0" />
       <mass
-        value="0.239419768320061" />
+        value="0.013" />
       <inertia
         ixx="0.000285938919722783"
@@ -296,5 +296,5 @@
 	<dynamics damping="50" friction="1"/>
   </joint>
-  <!--######################################################################-->
+  <!-- Link5 -->
   <link
     name="Link5">
@@ -304,12 +304,12 @@
         rpy="0 0 0" />
       <mass
-        value="0.218799761431678" />
-      <inertia
-        ixx="0.000350540363914072"
-        ixy="-3.41781619975602E-08"
-        ixz="-1.77056457224373E-08"
-        iyy="0.000104927867487581"
-        iyz="-7.82431228461971E-05"
-        izz="0.000334482418423629" />
+        value="0.013" />
+      <inertia
+        ixx="0.01"
+        ixy="0"
+        ixz="0"
+        iyy="0.01"
+        iyz="0"
+        izz="0.01" />
     </inertial>
     <visual>
@@ -356,5 +356,5 @@
 	<dynamics damping="50" friction="1"/>
   </joint>
-  <!--######################################################################-->
+  <!-- Link6 -->
   <link
     name="Link6">
@@ -364,12 +364,12 @@
         rpy="0 0 0" />
       <mass
-        value="0.0649018034311231" />
-      <inertia
-        ixx="2.02766547502765E-05"
-        ixy="-1.32505200276849E-06"
-        ixz="-2.5845091522508E-08"
-        iyy="1.87986725225022E-05"
-        iyz="3.39471452125439E-09"
-        izz="3.17885459163081E-05" />
+        value="0.013" />
+      <inertia
+        ixx="0.01"
+        ixy="0"
+        ixz="0"
+        iyy="0.01"
+        iyz="0"
+        izz="0.01" />
     </inertial>
     <visual>
@@ -414,10 +414,6 @@
       effort="10"
       velocity="3.92" />
-	<dynamics damping="50" friction="1"/>
-  </joint>
-  <!--######################################################################-->
-  <!-- This URDF was automatically created by SolidWorks to URDF Exporter! Originally created by Stephen Brawner (brawner@gmail.com)
-     Commit Version: 1.5.1-0-g916b5db  Build Version: 1.5.7152.31018
-     For more information, please see http://wiki.ros.org/sw_urdf_exporter -->
+    <dynamics damping="50" friction="1"/>
+  </joint>
   <!-- plate -->
   <link
@@ -426,19 +422,19 @@
       <origin
         xyz="0.04582 -2.25539999752262E-10 0.004046"
-        rpy="0 0 0" />
-      <mass
-        value="0.051308" />
-      <inertia
-        ixx="1.5915E-05"
-        ixy="2.51849999912398E-14"
-        ixz="1.4307E-07"
-        iyy="8.6534E-05"
-        iyz="4.91220000094025E-12"
-        izz="0.00010189" />
-    </inertial>
-    <visual>
-      <origin
-        xyz="0 0 0"
         rpy="1.5707963267949 0 0" />
+      <mass
+        value="0.013" />
+      <inertia
+        ixx="0.01"
+        ixy="0"
+        ixz="0"
+        iyy="0.01"
+        iyz="0"
+        izz="0.01" />
+    </inertial>
+    <visual>
+      <origin
+        xyz="0 0 0"
+        rpy="1.5707963267949 0 0" />
       <geometry>
         <mesh
@@ -454,5 +450,5 @@
       <origin
         xyz="0 0 0"
-        rpy="1.5707963267949 0 0" />
+        rpy="0 0 0" />
       <geometry>
         <mesh
@@ -473,10 +469,10 @@
     <dynamics damping="50" friction="1"/>
   </joint>
-  <!--######################################################################-->
-  <!-- realsense d435 with gazebo simulation    joint8 -->
+  <!-- realsense d435 with gazebo simulation    joint8
   <xacro:include filename="$(find realsense_ros_gazebo)/xacro/depthcam.xacro"/>
   <xacro:realsense_d435 sensor_name="d435" parent_link="plate" rate="10">
     <origin rpy="0 -1.5708 3.1416" xyz="0.08 0 0.0185"/>
   </xacro:realsense_d435>
+  -->
   <!--
   <xacro:arg name="use_nominal_extrinsics" default="false"/>
@@ -489,7 +485,5 @@
   </xacro:sensor_d435>
   -->
-  <!--######################################################################-->
   <!-- gripper -->
-  <!-- <xacro:include filename="$(find rm_65_description)/urdf/rm_65.gazebo.xacro"/> -->
   <xacro:include filename="$(find rm_65_description)/urdf/jawasm1.urdf.xacro" />
   <joint
@@ -505,5 +499,4 @@
     <dynamics damping="50" friction="1" />
   </joint>
-  <!--######################################################################-->
   <!-- Transmissions for ROS Control -->
   <xacro:macro name="transmission_block" params="joint_name" >
@@ -525,4 +518,6 @@
   <xacro:transmission_block joint_name="joint5"/>
   <xacro:transmission_block joint_name="joint6"/>
+  <xacro:transmission_block joint_name="joint7"/>
+  <xacro:transmission_block joint_name="joint9"/>
   <xacro:transmission_block joint_name="gripper_Link1"/>
   <xacro:transmission_block joint_name="gripper_Link2"/>
@@ -532,5 +527,5 @@
   <gazebo>
     <plugin name="gazebo_ros_control" filename="libgazebo_ros_control.so">
-      <robotNamespace>/</robotNamespace>
+      <robotNamespace>/arm</robotNamespace>
       <robotSimType>gazebo_ros_control/DefaultRobotHWSim</robotSimType>
       <legacyModeNS>true</legacyModeNS>

Commit message: before change

File: src/rm_robot/rm_65_description/urdf/jawasm1.urdf.xacro (robot description, xacro)
@@ -5,8 +5,8 @@
     <inertial>
       <origin
-        xyz="0.00339303654278191 -2.1205433560656E-05 -0.0099185365078758"
-        rpy="0 0 0" />
-      <mass
-        value="0.000001" />
+        xyz="0 0 0"
+        rpy="0 0 0" />
+      <mass
+        value="0.01" />
       <inertia
         ixx="3.93795927851199E-05"
@@ -41,4 +41,7 @@
     </collision>
   </link>
+  <gazebo reference="gripper_base_link">
+    <kinematic>1</kinematic>
+  </gazebo>
   <link
     name="gripper_Link1">
@@ -48,5 +51,5 @@
         rpy="0 0 0" />
       <mass
-        value="0.000001" />
+        value="0.01" />
       <inertia
         ixx="2.95068972140683E-07"
@@ -95,5 +98,5 @@
     <limit
       lower="0"
-      upper="1"
+      upper="0.1"
       effort="1"
       velocity="1" />
@@ -106,5 +109,5 @@
         rpy="0 0 0" />
       <mass
-        value="0.000001" />
+        value="0.01" />
       <inertia
         ixx="5.68538478020233E-07"
@@ -152,6 +155,6 @@
       xyz="0 0 1" />
     <limit
-      lower="-1"
-      upper="0"
+      lower="-0.1"
+      upper="0.1"
       effort="1"
       velocity="1" />
@@ -164,5 +167,5 @@
         rpy="0 0 0" />
       <mass
-        value="0.000001" />
+        value="0.01" />
       <inertia
         ixx="2.95068972140683E-07"
@@ -210,6 +213,6 @@
       xyz="0 0 1" />
     <limit
-      lower="-1"
-      upper="0"
+      lower="0"
+      upper="0.1"
       effort="1"
       velocity="1" />
@@ -222,5 +225,5 @@
         rpy="0 0 0" />
       <mass
-        value="0.000001" />
+        value="0.01" />
       <inertia
         ixx="5.68538478020238E-07"
@@ -268,6 +271,6 @@
       xyz="0 0 1" />
     <limit
-      lower="0"
-      upper="1"
+      lower="-0.1"
+      upper="0.1"
       effort="1"
       velocity="1" />

File: src/rm_robot/rm_65_description/urdf/rm_65.urdf.xacro (robot description, xacro)
@@ -13,5 +13,5 @@
         rpy="0 0 0" />
       <mass
-        value="14" />
+        value="140" />
       <inertia
         ixx="0.01"
@@ -51,4 +51,5 @@
     <kp value="100000000.0"/>
     <kd value="1.0"/>
+    <kinematic>1</kinematic>
   </gazebo>
   <joint name="dummy_joint" type="fixed">
@@ -114,6 +115,12 @@
       effort="60"
       velocity="3.14" />
-	<dynamics damping="50" friction="1"/>
-  </joint>
+  </joint>
+  <gazebo reference="link1">
+    <mu1 value="200000.0"/>
+    <mu2 value="200000.0"/>
+    <kp value="100000000.0"/>
+    <kd value="1.0"/>
+    <kinematic>1</kinematic>
+  </gazebo>
   <!-- Link2 -->
   <link
@@ -124,5 +131,5 @@
         rpy="0 0 0" />
       <mass
-        value="0.013" />
+        value="0.13" />
       <inertia
         ixx="0.00089150298478414"
@@ -184,5 +191,5 @@
         rpy="0 0 0" />
       <mass
-        value="0.013" />
+        value="0.13" />
       <inertia
         ixx="0.00063737100450158"
@@ -244,5 +251,5 @@
         rpy="0 0 0" />
       <mass
-        value="0.013" />
+        value="0.13" />
       <inertia
         ixx="0.000285938919722783"
@@ -304,12 +311,12 @@
         rpy="0 0 0" />
       <mass
-        value="0.013" />
-      <inertia
-        ixx="0.01"
-        ixy="0"
-        ixz="0"
-        iyy="0.01"
-        iyz="0"
-        izz="0.01" />
+        value="0.13" />
+      <inertia
+        ixx="0.000350540363914072"
+        ixy="-3.41781619975602E-08"
+        ixz="-1.77056457224373E-08"
+        iyy="0.000104927867487581"
+        iyz="-7.82431228461971E-05"
+        izz="0.000334482418423629" />
     </inertial>
     <visual>
@@ -364,11 +371,11 @@
         rpy="0 0 0" />
       <mass
-        value="0.013" />
+        value="0.13" />
       <inertia
         ixx="0.01"
-        ixy="0"
-        ixz="0"
+        ixy="0.01"
+        ixz="0.01"
         iyy="0.01"
-        iyz="0"
+        iyz="0.01"
         izz="0.01" />
     </inertial>
@@ -416,5 +423,5 @@
     <dynamics damping="50" friction="1"/>
   </joint>
-  <!-- plate -->
+  <!-- plate   -2.25539999752262E-10   -->
   <link
     name="plate">
@@ -422,7 +429,7 @@
       <origin
         xyz="0.04582 -2.25539999752262E-10 0.004046"
-        rpy="1.5707963267949 0 0" />
-      <mass
-        value="0.013" />
+        rpy="1.5708 0 0" />
+      <mass
+        value="0.01" />
       <inertia
         ixx="0.01"
@@ -436,5 +443,5 @@
       <origin
         xyz="0 0 0"
-        rpy="1.5707963267949 0 0" />
+        rpy="1.5708 0 0" />
       <geometry>
         <mesh
@@ -450,5 +457,5 @@
       <origin
         xyz="0 0 0"
-        rpy="0 0 0" />
+        rpy="1.5708 0 0" />
       <geometry>
         <mesh
@@ -458,21 +465,22 @@
   </link>
   <joint
-    name="joint7"
+    name="joint_plate"
     type="fixed">
     <origin
       xyz="0 0 0"
-      rpy="0 0 3.1416" />
+      rpy="0 0 3.1415" />
     <parent
       link="Link6" />
     <child
       link="plate" />
-    <dynamics damping="50" friction="1"/>
-  </joint>
-  <!-- realsense d435 with gazebo simulation    joint8
+  </joint>
+  <gazebo reference="plate">
+    <kinematic>1</kinematic>
+  </gazebo>
+  <!-- realsense d435 with gazebo simulation    joint8  -->
   <xacro:include filename="$(find realsense_ros_gazebo)/xacro/depthcam.xacro"/>
   <xacro:realsense_d435 sensor_name="d435" parent_link="plate" rate="10">
-    <origin rpy="0 -1.5708 3.1416" xyz="0.08 0 0.0185"/>
+    <origin rpy="0 -1.5708 3.1415" xyz="0.08 0 0.0185"/>
   </xacro:realsense_d435>
-  -->
   <!--
   <xacro:arg name="use_nominal_extrinsics" default="false"/>
@@ -499,5 +507,12 @@
     <dynamics damping="50" friction="1" />
   </joint>
-  <!-- Transmissions for ROS Control -->
+  <gazebo reference="gripper_base_link">
+    <mu1 value="200000.0"/>
+    <mu2 value="200000.0"/>
+    <kp value="100000000.0"/>
+    <kd value="1.0"/>
+    <kinematic>1</kinematic>
+  </gazebo>
+  <!--           Transmissions for ROS Control            -->
   <xacro:macro name="transmission_block" params="joint_name" >
     <transmission name="tran1">
@@ -518,6 +533,4 @@
   <xacro:transmission_block joint_name="joint5"/>
   <xacro:transmission_block joint_name="joint6"/>
-  <xacro:transmission_block joint_name="joint7"/>
-  <xacro:transmission_block joint_name="joint9"/>
   <xacro:transmission_block joint_name="gripper_Link1"/>
   <xacro:transmission_block joint_name="gripper_Link2"/>
@@ -533,3 +546,24 @@
   </gazebo>
   <!-- gazebo controller plugin for gripper -->
+  <gazebo>
+      <!-- loading plugin: mimic joints works in gazebo now -->
+      <plugin filename="libroboticsgroup_upatras_gazebo_mimic_joint_plugin.so" name="gripper_joint11_plugin">
+          <joint>gripper_Link1</joint>
+          <mimicJoint>gripper_Link11</mimicJoint>
+          <multiplier>1.0</multiplier>
+          <offset>0.0</offset>
+      </plugin>
+      <plugin filename="libroboticsgroup_upatras_gazebo_mimic_joint_plugin.so" name="gripper_joint2_plugin">
+          <joint>gripper_Link1</joint>
+          <mimicJoint>gripper_Link2</mimicJoint>
+          <multiplier>1.0</multiplier>
+          <offset>0.0</offset>
+      </plugin>
+      <plugin filename="libroboticsgroup_upatras_gazebo_mimic_joint_plugin.so" name="gripper_joint22_plugin">
+          <joint>gripper_Link1</joint>
+          <mimicJoint>gripper_Link22</mimicJoint>
+          <multiplier>1.0</multiplier>
+          <offset>0.0</offset>
+      </plugin>
+  </gazebo>
 </robot>
